File: esphome/kicad/chicken_coop/chicken_coop.kicad_pcb (KiCad board)
At the start: 2 copper layers, 3 parts, among them J1 Conn_01x04_Pin, U1 ESP32-CAM

Commit message: sync
Other:
- board outline added: 88.9 x 55.9 mm
Changed lines of the file:
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@@
     (pad "4" thru_hole circle (at 0 -13.208) (size 1.524 1.524) (drill 0.762) (layers "*.Cu" "*.Mask")
       (net 2 "GND") (pinfunction "GND_in") (pintype "input"))
-    (pad "5" thru_hole circle locked (at 18.542 -13.208) (size 1.524 1.524) (drill 0.762) (layers "*.Cu" "*.Mask")
+    (pad "5" thru_hole circle (at 18.542 -13.208) (size 1.524 1.524) (drill 0.762) (layers "*.Cu" "*.Mask")
       (net 2 "GND") (pinfunction "GND_Out") (pintype "output"))
     (pad "6" thru_hole circle (at 18.542 -10.668) (size 1.524 1.524) (drill 0.762) (layers "*.Cu" "*.Mask")
       (net 2 "GND") (pinfunction "GND_out") (pintype "input"))
-    (pad "7" thru_hole circle locked (at 18.542 -2.54) (size 1.524 1.524) (drill 0.762) (layers "*.Cu" "*.Mask")
+    (pad "7" thru_hole circle (at 18.542 -2.54) (size 1.524 1.524) (drill 0.762) (layers "*.Cu" "*.Mask")
       (net 1 "+5V") (pinfunction "Vcc_out") (pintype "input"))
     (pad "8" thru_hole circle (at 18.542 0.127) (size 1.524 1.524) (drill 0.762) (layers "*.Cu" "*.Mask")
@@
     )
   )
+  (gr_rect (start 88.9 33.02) (end 177.8 88.9)
+    (stroke (width 0.05) (type default)) (fill none) (layer "Edge.Cuts"))
   (segment (start 93.98 45.88) (end 93.98 40.64) (width 0.2) (layer "F.Cu") (net 2))
   (segment (start 107.569 38.1) (end 110.998 41.529) (width 0.2) (layer "F.Cu") (net 2))
