File: esphome/kicad/chicken_coop/chicken_coop.kicad_pcb (KiCad board)
At the start: 2 copper layers, 88.9 x 55.9 mm, 15 parts, among them J1 Conn_01x04_Pin, J2 Conn_01x04_Pin, J3 Conn_01x01_Pin, J4 Conn_01x02_Pin, U1 ESP32-CAM, U3 DRV8871 Module

Commit message: sync kicad
Parts:
- added D1: LED, LED_THT:LED_D4.0mm, F.Cu at (172.7, 73.7)
- added R3: 100K, Resistor_THT:R_Axial_DIN0207_L6.3mm_D2.5mm_P7.62mm_Horizontal, F.Cu at (186.7, 72.4)
Connections:
- U1 pad P$5: unconnected-(U1-IO15-PadP$5) -> STATUS
- U1 pad P$9: GND -> unconnected-(U1-.GND-PadP$9)
- U3 pad 1: IN2 -> GND
- U3 pad 2: IN1 -> +12V
- U3 pad 3: +12V -> IN1
- U3 pad 4: GND -> IN2
Routing:
- net STATUS: track 0.00 -> 23.4 mm
- net GND: track 187.6 -> 174.3 mm
- net +3.3V: track 84.7 -> 96.2 mm
- net Net-(D1-A): track 0.00 -> 4.34 mm
- net IN2: track 28.0 -> 30.1 mm
- net IN1: track 29.5 -> 31.6 mm
Other:
- board text added: "Lieven Merckx 2026-03-07 Chicken coop"
- board text removed: "Lieven Merckx 2026-02-13 Chicken coop"

Commit message: sync , 1k led res
Parts:
- R3: value 100K -> 1K
