File: esphome/kicad/chicken_coop/chicken_coop.kicad_sch (KiCad schematic)
At the start: 11 parts, among them J1 Conn_01x04_Pin, J2 Conn_01x04_Pin, J3 Conn_01x01_Pin, J4 Conn_01x02_Pin, U1 ESP32-CAM, U3 DRV8871 Module

Commit message: sync kicad
Parts:
- added D1: LED, LED_THT:LED_D4.0mm, symbol Device:LED
- added R3: 100K, Resistor_THT:R_Axial_DIN0207_L6.3mm_D2.5mm_P7.62mm_Horizontal, symbol Device:R
Connections:
- net +12V: now also U3.2 (VM); no longer U3.3 (VM)
- net +3.3V: now also R3.1
- net GND: now also U3.1 (GND); no longer U1.P$9 (.GND), U3.4 (GND)
- net IN1: now also U3.3 (IN1); no longer U3.2 (IN1)
- net IN2: now also U3.4 (IN2); no longer U3.1 (IN2)
- net STATUS: now reaches U1.P$5 (IO15)
- net STATUS: now also D1.1 (K)
- new net: D1.2 (A), R3.2
Changed lines of the file:
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@@
+    (stroke (width 0) (type default))
+  )
+  (wire (pts (xy 245.11 138.43) (xy 252.73 138.43))
     (stroke (width 0) (type default))
   )
@@
     (stroke (width 0) (type default))
   )
+  (wire (pts (xy 252.73 113.03) (xy 252.73 116.84))
+    (stroke (width 0) (type default))
+  )
   (wire (pts (xy 80.01 135.89) (xy 104.14 135.89))
     (stroke (width 0) (type default))
@@
     (stroke (width 0) (type default))
   )
+  (wire (pts (xy 252.73 138.43) (xy 252.73 135.89))
+    (stroke (width 0) (type default))
+  )
   (wire (pts (xy 215.9 102.87) (xy 198.12 102.87))
     (stroke (width 0) (type default))
@@
     (stroke (width 0) (type default))
   )
-  (wire (pts (xy 198.12 107.95) (xy 205.74 107.95))
+  (wire (pts (xy 163.83 100.33) (xy 167.64 100.33))
     (stroke (width 0) (type default))
   )
@@
   )
   (wire (pts (xy 57.15 49.53) (xy 57.15 52.07))
+    (stroke (width 0) (type default))
+  )
+  (wire (pts (xy 252.73 124.46) (xy 252.73 128.27))
     (stroke (width 0) (type default))
   )
@@
     )
   )
+  (global_label "STATUS" (shape input) (at 163.83 100.33 180) (fields_autoplaced)
+    (effects (font (size 1.27 1.27)) (justify right))
+    (property "Intersheetrefs" "${INTERSHEET_REFS}" (at 154.0715 100.33 0)
+      (effects (font (size 1.27 1.27)) (justify right) hide)
+    )
+  )
+  (global_label "STATUS" (shape input) (at 245.11 138.43 180) (fields_autoplaced)
+    (effects (font (size 1.27 1.27)) (justify right))
+    (property "Intersheetrefs" "${INTERSHEET_REFS}" (at 235.3515 138.43 0)
+      (effects (font (size 1.27 1.27)) (justify right) hide)
+    )
+  )
   (global_label "IN1" (shape input) (at 162.56 95.25 180) (fields_autoplaced)
     (effects (font (size 1.27 1.27)) (justify right))
@@
         (path "/1849e995-fa12-415f-a5e1-2f1ea65d51ac"
           (reference "#PWR013") (unit 1)
+        )
+      )
+    )
+  )
+  (symbol (lib_id "Device:R") (at 252.73 120.65 0) (unit 1)
+    (in_bom yes) (on_board yes) (dnp no) (fields_autoplaced)
+    (property "Reference" "R3" (at 255.27 119.38 0)
+      (effects (font (size 1.27 1.27)) (justify left))
+    )
+    (property "Value" "100K" (at 255.27 121.92 0)
+      (effects (font (size 1.27 1.27)) (justify left))
+    )
+    (property "Footprint" "Resistor_THT:R_Axial_DIN0207_L6.3mm_D2.5mm_P7.62mm_Horizontal" (at 250.952 120.65 90)
+      (effects (font (size 1.27 1.27)) hide)
+    )
+    (property "Datasheet" "~" (at 252.73 120.65 0)
+      (effects (font (size 1.27 1.27)) hide)
+    )
+    (pin "1")
+    (pin "2")
+    (instances
+      (project "chicken_coop"
+        (path "/1849e995-fa12-415f-a5e1-2f1ea65d51ac"
+          (reference "R3") (unit 1)
         )
       )
@@
     )
   )
+  (symbol (lib_id "power:+3.3V") (at 252.73 113.03 0) (unit 1)
+    (in_bom yes) (on_board yes) (dnp no)
+    (property "Reference" "#PWR018" (at 252.73 116.84 0)
+      (effects (font (size 1.27 1.27)) hide)
+    )
+    (property "Value" "+3.3V" (at 255.27 110.49 0)
+      (effects (font (size 1.27 1.27)))
+    )
+    (property "Footprint" "" (at 252.73 113.03 0)
+      (effects (font (size 1.27 1.27)) hide)
+    )
+    (property "Datasheet" "" (at 252.73 113.03 0)
+      (effects (font (size 1.27 1.27)) hide)
+    )
+    (pin "1")
+    (instances
+      (project "chicken_coop"
+        (path "/1849e995-fa12-415f-a5e1-2f1ea65d51ac"
+          (reference "#PWR018") (unit 1)
+        )
+      )
+    )
+  )
   (symbol (lib_id "power:+3.3V") (at 246.38 43.18 0) (unit 1)
     (in_bom yes) (on_board yes) (dnp no) (fields_autoplaced)
@@
     )
   )
-  (symbol (lib_id "power:GND") (at 205.74 107.95 0) (unit 1)
-    (in_bom yes) (on_board yes) (dnp no) (fields_autoplaced)
-    (property "Reference" "#PWR03" (at 205.74 114.3 0)
-      (effects (font (size 1.27 1.27)) hide)
-    )
-    (property "Value" "GND" (at 205.74 113.03 0)
-      (effects (font (size 1.27 1.27)))
-    )
-    (property "Footprint" "" (at 205.74 107.95 0)
-      (effects (font (size 1.27 1.27)) hide)
-    )
-    (property "Datasheet" "" (at 205.74 107.95 0)
-      (effects (font (size 1.27 1.27)) hide)
-    )
-    (pin "1")
-    (instances
-      (project "chicken_coop"
-        (path "/1849e995-fa12-415f-a5e1-2f1ea65d51ac"
-          (reference "#PWR03") (unit 1)
-        )
-      )
-    )
-  )
   (symbol (lib_id "power:GND") (at 207.01 96.52 0) (unit 1)
     (in_bom yes) (on_board yes) (dnp no)
@@
         )
       )
+    )
+  )
+  (symbol (lib_id "Device:LED") (at 252.73 132.08 90) (unit 1)
+    (in_bom yes) (on_board yes) (dnp no) (fields_autoplaced)
+    (property "Reference" "D1" (at 256.54 132.3975 90)
+      (effects (font (size 1.27 1.27)) (justify right))
+    )
+    (property "Value" "LED" (at 256.54 134.9375 90)
+      (effects (font (size 1.27 1.27)) (justify right))
+    )
+    (property "Footprint" "LED_THT:LED_D4.0mm" (at 252.73 132.08 0)
+      (effects (font (size 1.27 1.27)) hide)
+    )
+    (property "Datasheet" "~" (at 252.73 132.08 0)
+      (effects (font (size 1.27 1.27)) hide)
+    )
+    (pin "1")
+    (pin "2")
+    (instances
+      (project "chicken_coop"
+        (path "/1849e995-fa12-415f-a5e1-2f1ea65d51ac"
+          (reference "D1") (unit 1)
+        )
+      )

Commit message: sync , 1k led res
Parts:
- R3: value 100K -> 1K
